File: blinkrad ledboard/ledboard_noISP.sch (EAGLE design)
At the start: 17 parts, among them IC1 TINY13-20SSU

Commit message: MASSIVE ERROR, USE N FET
Parts:
- Q-BLUE, Q-GREEN, Q-RED: device SparkFun-DiscreteSemi:MOSFET-PCHANNELDMG2307L -> SparkFun-DiscreteSemi:MOSFET-NCHANNELBSS123LT1G
Changed lines of the file:
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@@
 <parts>
 <part name="D1" library="SparkFun-LED" deviceset="LED-RGB-CA-THRU" device="CLEAR"/>
-<part name="Q-RED" library="SparkFun-DiscreteSemi" deviceset="MOSFET-PCHANNEL" device="DMG2307L" value="30V, 2.5A"/>
-<part name="Q-GREEN" library="SparkFun-DiscreteSemi" deviceset="MOSFET-PCHANNEL" device="DMG2307L" value="30V, 2.5A"/>
-<part name="Q-BLUE" library="SparkFun-DiscreteSemi" deviceset="MOSFET-PCHANNEL" device="DMG2307L" value="30V, 2.5A"/>
+<part name="Q-RED" library="SparkFun-DiscreteSemi" deviceset="MOSFET-NCHANNEL" device="BSS123LT1G" value="30V, 2.5A"/>
+<part name="Q-GREEN" library="SparkFun-DiscreteSemi" deviceset="MOSFET-NCHANNEL" device="BSS123LT1G" value="30V, 2.5A"/>
+<part name="Q-BLUE" library="SparkFun-DiscreteSemi" deviceset="MOSFET-NCHANNEL" device="BSS123LT1G" value="30V, 2.5A"/>
 <part name="R-RED" library="SparkFun-Resistors" deviceset="RESISTOR" device="0603"/>
 <part name="R-GREEN" library="SparkFun-Resistors" deviceset="RESISTOR" device="0603"/>
